File: afm_saucer_pcb/afm_saucer/afm_saucer.kicad_pcb (KiCad board)
At the start: 2 copper layers, 120.1 x 118.9 mm, 42 parts, among them J1 Conn_01x08_Male, J2 Conn_01x02_Male, J3 Conn_02x03_Odd_Even, SW1 Vibration Sensor, SW2 SW_Push, SW3 SW_DIP_x04, U1 OKI-78SR-5_1.5-W36-C, U2 ATmega328P-P, Y1 Crystal

Commit message: PCB v1.1
Parts:
- added G***: LOGO, bfl:qrcode, B.Cu at (67.0, 82.1)
- QR: renamed from G***; value LOGO -> QRCODE
- moved G*** 51.1 mm to (142.9, 88.7)
- moved SW1 47.2 mm to (135.0, 73.7), turned to 42 degrees
Routing:
- net Net-(R5-Pad1): track 25.4 -> 73.2 mm
- net GND: track 692.4 -> 708.4 mm
Other:
- board text added: "v1.1"
- board text removed: "v1.0"
